File: Hardware/lora minimo.sch (KiCad schematic (older format))
At the start: 38 parts, among them J1 USB_B, J2 Conn_01x03, J3 Conn_01x04, SW1 SW_Push, U1 ATSAMD21E18A-MU, U2 MCP73831-2-OT, U3 AP2112K-3.3, U4 RFM95W-868S2

Commit message: ACELEROMETER AND EPROOM
Parts:
- removed D2: LED, symbol device:LED
- removed R?: R, symbol device:R
- added C11: 4.7 uF, symbol device:C
- added C12: 10uF, symbol device:C
- added C13, C15, C17: 0.1 uF, Capacitors_SMD:C_0805_HandSoldering, symbol device:C
- added C14: 0.01 uF, symbol device:C
- added C16: 2200 pF, symbol device:C
- added D7: LED_Small_ALT, symbol device:LED_Small_ALT
- added H1, H2, H3, H4: MountingHole, symbol Mechanical:MountingHole
- added Q3: 2N2219, Package_TO_SOT_THT:TO-39-3, symbol Transistor_BJT:2N2219
- added R10, R9: 120, symbol device:R
- added R11, R13: 10K, symbol device:R
- added R12: 10 K, symbol device:R
- added R14, R15: 10 K, symbol device:R_Small
- added R16: 1k, symbol device:R
- added R17: 4.7 K, symbol device:R
- added R7: 1.2K, symbol device:R
- added R8: 1.2 K, symbol device:R
- added U5: 24LC256, Housings_SOIC:SOIC-8_3.9x4.9mm_Pitch1.27mm, symbol memory:24LC256
- added U6: AP2112K-3.3, Package_TO_SOT_SMD:SOT-23-5, symbol Regulator_Linear:AP2112K-3.3
- added U7: MPU-6050, symbol sensors:MPU-6050
- C1, C10: footprint (none) -> Capacitors_SMD:C_0805_HandSoldering; manf# (none) -> 885012207072
- C2: value C -> 1uF; footprint (none) -> Capacitors_SMD:C_0805_HandSoldering; manf# (none) -> GRM21BC80J106KE19L
- C3: value C -> 0.1 uF; footprint (none) -> Capacitors_SMD:C_0805_HandSoldering; manf# (none) -> 885012207072
- C4, CIN1: value C -> 4.7 uF
- D4: manf# (none) -> APT2012SGC
- D6: manf# (none) -> AP2012EC
- J1: footprint (none) -> USB:629004113921
- R1, R3: value R -> 100 K
- R2: value R -> 2 K
- R4, R5: renamed from R?; value R -> 10 K
- RLED1: value R -> 120; manf# (none) -> RMC1/10K1200FTP
- SW1: manf# (none) -> B3U-1000P
- U1: manf# (none) -> ATSAMD21E15B-AUT
- U3: manf# (none) -> AP2114H-3.3TRG1
- gave numbers to parts that had none: 5
Connections:
- net BATT+ is gone; now on net VBUS: BT1.1 (+), C4.1, C8.1, D3.1 (K), Q2.2 (E), R1.1, U2.3 (VBAT), U3.1 (VIN)
- net 1PPS: now also U1.22 (PA23)
- net ADCX: now also U1.5 (PA04)
- net DI3: no longer U1.1 (PA00)
- net DIO0: no longer U1.5 (PA04)
- net DIO1: no longer U1.22 (PA23)
- net DO2: no longer U1.7 (PA06)
- net DO3: no longer U1.6 (PA05)
- net GND: now also Q1.1 (S), R4.2, C11.2, C12.2, C13.2, C14.1, C15.2, C17.2, Q3.1 (E), R10.2, R12.2, R17.1, R9.2, U5.1 (A0), U5.2 (A1), U5.3 (A2), U5.4 (GND), U6.2 (GND), U7.1 (CLKIN), U7.11 (FSYNC); no longer D4.1 (K), D5.1 (K)
- net STAT: now also RLED1.2
- net VBUS: now also C11.1, R11.1, R13.1, R7.2, R8.2, U5.8 (VCC), U6.1 (VIN); no longer RLED1.1
- net at D6.1 (K): now also RLED1.1
- new net: D4.1 (K), R9.1
- new net: D5.1 (K), R10.1
- new net: Q3.2 (B), R7.1
- new net: C15.1, U7.10 (REGOUT)
- new net: C16.2, U7.18 (GND)
- new net: C16.1, U7.20 (CPOUT)
- new net: R17.2, U7.9 (AD0)
- new net: D7.2 (A), R16.2
- new net: R12.1, U5.7 (WP)
- new net 3.3VoltsMPU: C12.1, C13.1, C14.2, C17.1, R14.2, R15.1, R16.1, U6.5 (VOUT), U7.13 (VDD), U7.8 (VDDIO)
- new net DIG-IO: Q3.3 (C), R8.1, U1.1 (PA00)
- new net INT: U7.12 (INT)
- new net SCL: R13.2, R15.2, U1.7 (PA06), U5.6 (SCL), U7.23 (SCL)
- new net SDA: R11.2, R14.1, U1.6 (PA05), U5.5 (SDA), U7.24 (SDA)
- new net XCL: U7.7 (AUX_SCL)
- new net XDA: U7.6 (AUX_SDA)
- no-connect marks 7 -> 8
Other:
- note added: "ACELEROMETER\n"
- note added: "BYPASS\n"
- note added: "COMM\n\n"
- note added: "FALTA SEÑALAR LA MANUFACTURA DEL DIODO, FUSIBLE Y USB\n"
- note added: "LOGO\n"
- note added: "MOUNTING-HOLE\n"
- note added: "REGULATOR AND CHARGE\n\n"
- note added: "\n EPROOM\n"
- note removed: "COMUNICACION\n"
- moved on the sheet: BT1, C5, C6, C7, CIN1, D3, D4, D5, D6, MODULE1, Q1, Q2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

Commit message: MEMORY AND ACCELEROMETER UPDATE
CHANGED BY A FLASH MEMORY OF 2 MB AND CHANGED BY ACCELEROMETER MODULE
Parts:
- removed C11: 4.7 uF, symbol device:C
- removed C12: 10uF, symbol device:C
- removed C13, C15, C17: 0.1 uF, Capacitors_SMD:C_0805_HandSoldering, symbol device:C
- removed C14: 0.01 uF, symbol device:C
- removed C16: 2200 pF, symbol device:C
- removed D7: LED_Small_ALT, symbol device:LED_Small_ALT
- removed J2: Conn_01x03, symbol conn:Conn_01x03
- removed Q3: 2N2219, Package_TO_SOT_THT:TO-39-3, symbol Transistor_BJT:2N2219
- removed R14, R15: 10 K, symbol device:R_Small
- removed R16: 1k, symbol device:R
- removed R17: 4.7 K, symbol device:R
- removed R7: 1.2K, symbol device:R
- removed R8: 1.2 K, symbol device:R
- removed U6: AP2112K-3.3, Package_TO_SOT_SMD:SOT-23-5, symbol Regulator_Linear:AP2112K-3.3
- removed U7: MPU-6050, symbol sensors:MPU-6050
- added C11: 0.1uF, symbol device:C_Small
- added J2: Conn_01x08, symbol conn:Conn_01x08
- added U6: W25Q16BVSSIG, SOIC127P790X216-8N, symbol electroniccats:W25Q16BVSSIG
- AE1: value Antenna_Shield -> Antenna_Shiel
- C4, C8, C9, CIN1: manf# (none) -> GRT21BR61H475KE13L
- C5: manf# (none) -> 885012207072
- C6: manf# (none) -> 885012207072; manf#  (none) -> 885012207072
- C7: manf# (none) -> GRM21BC80J106KE19L
- D1: manf# (none) -> 1N5819HW-7-F
- D5: manf# (none) -> SML-LXF0805SYC-TR
- D6: manf# AP2012EC -> AP2012EC
- F1: manf# (none) -> MF-MSMF050-2
- J1: manf# (none) -> 629105150521
- R1, R3: manf# (none) -> SG73G2ATTD1003D
- R11, R12, R13, R4, R5: manf# (none) -> SG73G2ATTD1002D
- R2: manf# (none) -> KTR10EZPJ102
- U2: manf# (none) -> MCP73831T-2ATI/OT
- U5: manf# (none) -> 24LC256-I/SN
Connections:
- net RX is gone; now on net Rx: MODULE1.1 (RXD), U1.14 (PA11)
- net +3V3: now also C11.1, J2.7 (Pin_7), U6.8 (VCC)
- net 1PPS: no longer D5.2 (A)
- net GND: now also C11.2, J2.6 (Pin_6), U6.4 (GND)
- net MISO: now also U6.2 (DO(IO1))
- net MOSI: now also U6.5 (DI(IO0))
- net SCK: now also U6.6 (CLK)
- net SCL: now also J2.5 (Pin_5)
- net SDA: now also J2.4 (Pin_4)
- net VBUS: now also J2.8 (Pin_8)
- net FLASH_HD: now reaches U1.11 (PA08)
- net FLASH_HD: now also U6.7 (/HOLD(IO3))
- net FLASH_WP: now reaches U1.12 (PA09)
- net FLASH_WP: now also U6.3 (/WP(IO2))
- net DI1: no longer names the net of U1.3 (PA02)
- net DI2: no longer names the net of U1.2 (PA01)
- net DIG-IO: no longer names the net of U1.1 (PA00)
- net DO1 renamed FLASH_CS
- net FLASH_CS: now also U6.1 (/CS)
Other:
- note added: "COM\n"
- note added: "EPROOM\n"
- note added: "FLASH\n"
- note added: "INDICATOR LEDS\n"
- note added: "RFM95W"
- note removed: "ANTENA\n"
- note removed: "COMM\n\n"
- note removed: "FALTA SEÑALAR LA MANUFACTURA DEL DIODO, FUSIBLE Y USB\n"
- note removed: "\n EPROOM\n"
- moved on the sheet: AE1, C3, C5, C6, C7, D1, D4, D5, D6, F1, J1, J3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

Commit message: connection update
Parts:
- removed D1: D_Schottky, symbol device:D_Schottky
- removed U3: AP2112K-3.3, Package_TO_SOT_SMD:SOT-23-5, symbol Regulator_Linear:AP2112K-3.3
- added U3: AP2114H-3.3TRG1, TO_SOT_Packages_SMD:SOT-223-3Lead_TabPin2, symbol agroin:AP2114H-3.3TRG1
- MODULE1: footprint QUECTEL_L80-M39 -> Rf:QUECTEL_L80-M39
Connections:
- net +3V3: now also C9.1, U3.2 (OUT)
- net DIO0: now also U1.1 (PA00)
- net DIO1: now also U1.2 (PA01)
- net DIO2: now also U1.3 (PA02); no longer U1.25 (PA27)
- net GND: now also U3.1 (GND); no longer BT1.2 (-), Q1.3 (D), R5.2
- net VBUS: now also F1.2; no longer BT1.1 (+), C4.1, C8.1, D3.1 (K), Q2.2 (E), R1.1, U2.3 (VBAT)
- new net: BT1.2 (-), Q1.3 (D), R5.2
- new net +BATT: BT1.1 (+), C4.1, C8.1, D3.1 (K), Q2.2 (E), U3.3 (IN)
- new net VBAT: R1.1, U2.3 (VBAT)
- no-connect marks 8 -> 12
Other:
- moved on the sheet: C1, C4, C9, CIN1, J3

Commit message: add netist and pcb
Parts:
- removed R11, R13: 10K, symbol device:R
- removed R12: 10 K, symbol device:R
- removed U5: 24LC256, Housings_SOIC:SOIC-8_3.9x4.9mm_Pitch1.27mm, symbol memory:24LC256
- AE1: footprint (none) -> Rf:SMA_EDGE
- BT1: footprint (none) -> Batteries:BAT-HLD-012-SMT-OTL
- C11: footprint (none) -> Capacitors_SMD:C_0805_HandSoldering; manf# (none) -> 885012207072
- C4, C5, C7, C8, C9, CIN1: footprint (none) -> Capacitors_SMD:C_0805_HandSoldering
- C6: footprint (none) -> Capacitors_SMD:C_0805_HandSoldering; manf#  885012207072 -> (none)
- D3: footprint Diode_THT:D_DO-35_SOD27_P7.62mm_Horizontal -> Diodes_SMD:D_SOD-323_HandSoldering; manf# (none) -> 512-1N4148WS
- D4, D5, D6: footprint (none) -> LEDs:LED_0805_HandSoldering
- F1: footprint (none) -> Resistors_SMD:R_1812_HandSoldering
- H1, H2, H3, H4: footprint (none) -> Mounting_Holes:MountingHole_3.2mm_M3_Pad_Via
- J1: footprint USB:629004113921 -> USB_WURTH:629105150521
- J2: footprint (none) -> Pin_Headers:Pin_Header_Straight_1x08_Pitch2.54mm
- J3: footprint (none) -> Pin_Headers:Pin_Header_Straight_1x04_Pitch2.54mm
- Q1: value 2N7000 -> 2N7002; footprint Package_TO_SOT_THT:TO-92_Inline -> TO_SOT_Packages_SMD:SOT-23; manf# (none) -> 512-2N7002
- Q2: footprint (none) -> TO_SOT_Packages_SMD:SOT-23; manf# (none) -> MMBT3904LT3G newark
- R1, R10, R2, R3, R4, R5, R9, RLED1: footprint (none) -> Resistors_SMD:R_0805_HandSoldering
- SW1: footprint (none) -> Buttons_Switches_SMD:SW_SPST_B3U-1000P-B
- U1: footprint QFN50P500X500X100-33N -> Housings_QFP:TQFP-48_7x7mm_Pitch0.5mm
- U2: footprint Package_TO_SOT_SMD:SOT-23-5 -> TO_SOT_Packages_SMD:SOT-23-5_HandSoldering
- U3: footprint TO_SOT_Packages_SMD:SOT-223-3Lead_TabPin2 -> TO_SOT_Packages_SMD:SOT-223; manf# (none) -> AP2114H-3.3TRG1
- U4: footprint (none) -> Rf:RFM95W
- U6: footprint SOIC127P790X216-8N -> Housings_SOIC:Diodes_PSOP-8
Other:
- note removed: "EPROOM\n"

Commit message: PCB test
pcb design and fingerprint reallocation
Parts:
- AE1: footprint Rf:SMA_EDGE -> Rf:AMPHENOL_901-144
- H1, H2, H3, H4: footprint Mounting_Holes:MountingHole_3.2mm_M3_Pad_Via -> Mounting_Holes:MountingHole_5.3mm_M5_Pad_Via
- J1: footprint USB_WURTH:629105150521 -> Connectors_ec:629105150521
- J2: value Conn_01x08 -> Acelerometer
- J3: value Conn_01x04 -> SWD; footprint Pin_Headers:Pin_Header_Straight_1x04_Pitch2.54mm -> Pin_Headers:Pin_Header_Straight_2x02_Pitch2.54mm
- SW1: value SW_Push -> RESET
- U1: footprint Housings_QFP:TQFP-48_7x7mm_Pitch0.5mm -> Housings_QFP:TQFP-32_7x7mm_Pitch0.8mm
- U3: footprint TO_SOT_Packages_SMD:SOT-223 -> TO_SOT_Packages_SMD:SOT-223-3_TabPin2
- renumbered CIN1 to C12
Connections:
- net 1PPS: now also D5.2 (A)
- no-connect marks 12 -> 11
Other:
- moved on the sheet: BT1, C11, C12, C4, C5, C6, C7, C8, C9, D3, D4, D5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
