File: gps_lora/gps_minimo/gps_minimo.sch (KiCad schematic (older format))
At the start: 18 parts, among them J1 USB_B, J2 BAT, Q1 Q_PMOS_GSD, U1 AP2114-3.3, U2 MCP73831-3-OT

Commit message: add pcb gps vehicular and minimo
Changed lines of the file:
@@
 EESchema Schematic File Version 4
 LIBS:gps_minimo-cache
-EELAYER 26 0
+EELAYER 29 0
 EELAYER END
 $Descr A4 11693 8268
@@
 	3540 1970 3600 1970
 Wire Wire Line
-	4210 1970 4210 1770
-Wire Wire Line
 	3140 2570 3140 2630
 Wire Wire Line
@@
 	3500 4090 3500 4450
 Wire Wire Line
-	3500 5130 3740 5130
-Wire Wire Line
 	3500 5390 3500 5130
 Connection ~ 3500 5130
@@
 	4320 4650 4320 5130
 Connection ~ 4320 5130
-Wire Wire Line
-	4320 5130 4580 5130
 Wire Wire Line
 	4320 5420 4320 5130
@@
 Wire Wire Line
 	3900 1970 4210 1970
+Wire Wire Line
+	4210 1770 4210 1970
+Wire Wire Line
+	4580 5130 4320 5130
+Wire Wire Line
+	4040 5130 4320 5130
+Wire Wire Line
+	3500 5130 3740 5130
 $Comp
 L Device:D_Schottky D2
@@
 	-1   0    0    1
 $EndComp
-Wire Wire Line
-	4040 5130 4320 5130
 $EndSCHEMATC
