File: gps_lora/gps_minimo/microcontroller.sch (KiCad schematic (older format))
At the start: 12 parts, among them J3 SWD, SW1 RST, U3 ATSAMD21E, U4 RFM95W-868S2

Commit message: add pcb gps vehicular and minimo
Parts:
- U3: symbol gps_LoRa:ATSAMD21E -> gps_minimo-rescue:ATSAMD21E-gps_LoRa
- U4: symbol gps_LoRa:RFM95W-868S2 -> gps_minimo-rescue:RFM95W-868S2-gps_LoRa
Connections:
- net 1PPS: now also U3.15 (PA14/I14/SERCOM2+4.2)
- net LED_1: now also U3.1 (PA00/EINT0/SERCOM1.0)
- net LED_2: now also U3.2 (PA01/EINT1/SERCOM1.1)
- net V_DIV: now reaches U3.3 (PA02/EINT2/AIN0/Y0/VOUT)
- no-connect marks 6 -> 13
Changed lines of the file:
@@
 EESchema Schematic File Version 4
 LIBS:gps_minimo-cache
-EELAYER 26 0
+EELAYER 29 0
 EELAYER END
 $Descr A4 11693 8268
@@
 $EndComp
 $Comp
-L gps_LoRa:ATSAMD21E U3
+L gps_minimo-rescue:ATSAMD21E-gps_LoRa U3
 U 1 1 5C7B383C
 P 4900 3340
@@
 $EndComp
 $Comp
-L gps_LoRa:RFM95W-868S2 U4
+L gps_minimo-rescue:RFM95W-868S2-gps_LoRa U4
 U 1 1 5C7B3DA5
 P 9220 4540
@@
 	9680 2950 9680 3100
 Connection ~ 9680 3100
+Text Label 6300 1740 0    50   ~ 0
+LED_1
+Text Label 6300 1840 0    50   ~ 0
+LED_2
+Text GLabel 6300 1940 2    50   Input ~ 0
+V_DIV
+Text Label 6300 3340 0    50   ~ 0
+1PPS
+NoConn ~ 6300 2040
+NoConn ~ 6300 2240
+NoConn ~ 6300 2340
+NoConn ~ 6300 2440
+NoConn ~ 6300 2640
+NoConn ~ 6300 2740
+NoConn ~ 6300 4740
 $EndSCHEMATC
