File: gps_lora/gps_vehicular/microcontroller.sch (KiCad schematic (older format))
At the start: 30 parts, among them J5 IGN, J6 RELAY, J7 PANI, J8 SWD, Q2 SMMBT3904LT1G, Q3 SMMBT3904LT1G, SW1 RST, U4 LTV-352T, U5 LTV-352T, U6 ATSAMD21E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

Commit message: add pcb gps vehicular and minimo
Parts:
- MODULE1: symbol electroniccats:L80-M39 -> gps_vehicular-rescue:L80-M39-electroniccats
Connections:
- net 1PPS: now also U6.15 (PA14/I14/SERCOM2+4.2)
- net LED_1: now also U6.1 (PA00/EINT0/SERCOM1.0)
- net LED_2: now also U6.2 (PA01/EINT1/SERCOM1.1)
- net OUT_SIG: now also U6.8 (PA07/I7/AIN7/SERCOM0.3/I2SD0)
- net SIG_CONECTADO: now also U6.6 (PA05/EINT5/AIN5/SERCOM0.1)
- net SIG_IGNI: now also U6.7 (PA06/EINT6/AIN6/SERCOM0.2)
- net SIG_PANI: now also U6.12 (PA09/I2C/I9/AIN17/SERCOM0+2.1/I2SMC)
- no-connect marks 6 -> 9
Changed lines of the file:
@@
 EESchema Schematic File Version 4
 LIBS:gps_vehicular-cache
-EELAYER 26 0
+EELAYER 29 0
 EELAYER END
 $Descr A4 11693 8268
@@
 $EndComp
 $Comp
-L electroniccats:L80-M39 MODULE1
+L gps_vehicular-rescue:L80-M39-electroniccats MODULE1
 U 1 1 5C6B22A1
 P 9030 1590
@@
 	9690 2090 9690 2190
 Connection ~ 9690 2190
+Text Label 6300 2410 0    50   ~ 0
+1PPS
+Text Label 6300 810  0    50   ~ 0
+LED_1
+Text Label 6300 910  0    50   ~ 0
+LED_2
+Text Label 6300 1410 0    50   ~ 0
+SIG_IGNI
+Text Label 6300 1510 0    50   ~ 0
+OUT_SIG
+Text Label 6300 1810 0    50   ~ 0
+SIG_PANI
+Text Label 6300 1310 0    50   ~ 0
+SIG_CONECTADO
+NoConn ~ 6300 1110
+NoConn ~ 6300 1710
+NoConn ~ 6300 3810
 $EndSCHEMATC
